Commit message: Added the moveit pos program and workspace env

File: mycobot_pro_600_desp/urdf/mycobot_pro_600.urdf (robot description, URDF)
Before this commit: robot mycobot_600, 7 links, 6 joints
Links:
- added link env_world; visual mesh filename=package://mycobot_pro_600_desp/urdf/suit_env_v2.dae
Joints:
- added joint env_world_fixed_joint: type fixed, parent base, child env_world, origin xyz=0.3 0.2 0 rpy=0 0 0

Commit message: Trajectory Planning Successful but joit states unpublished with few changes to the urdf

File: mycobot_pro_600_desp/urdf/mycobot_pro_600.urdf (robot description, URDF)
Before this commit: robot mycobot_600, 8 links, 7 joints
Joints:
- joint joint3_to_joint2: limit lower=-4.7123 upper=1.5708 effort=30.0 velocity=3.0 -> lower=-3.57792 upper=0.418879 effort=30.0 velocity=3.0
- joint joint4_to_joint3: limit lower=-2.6179 upper=2.443 effort=30.0 velocity=3.0 -> lower=-2.0944 upper=2.443 effort=30.0 velocity=3.0
- joint joint5_to_joint4: limit lower=-4.5378 upper=1.3962 effort=30.0 velocity=3.0 -> lower=-3.14159 upper=1.3962 effort=30.0 velocity=3.0
- joint joint6_to_joint5: limit lower=-2.9321 upper=2.9321 effort=1000.0 velocity=3.0 -> lower=-3.14 upper=3.14 effort=1000.0 velocity=3.0

Commit message: Prithvi (#7)
* changed trajectory

* basics are working need to work on robotstate

* Removed unwanted packages

File: mycobot_pro_600_desp/urdf/mycobot_pro_600.urdf (robot description, URDF)
Before this commit: robot mycobot_600, 8 links, 7 joints
Joints:
- joint env_world_fixed_joint: origin xyz=0.3 0.2 0 rpy=0 0 0 -> xyz=-0.15 -0.25 0 rpy=0 0 3.14159
- joint joint3_to_joint2: limit lower=-4.7123 upper=1.5708 effort=30.0 velocity=3.0 -> lower=-3.14 upper=0 effort=30.0 velocity=3.0
