Commit message: Fixed MovitConfig and oreientatiosn

File: mycobot_pro_600_description/urdf/mycobot_pro_600.urdf (robot description, URDF)
Before this commit: robot firefighter, 7 links, 6 joints
Links:
- added link endEffector
- added link env_world; visual mesh filename=package://mycobot_pro_600_description/urdf/suit_env_v2.dae
- link base: geometry collision mesh filename=package://mycobot_pro_600_description/urdf/base.dae; visual mesh filename=package://mycobot_pro_600_description/urdf/base.dae
- link link1: geometry collision mesh filename=package://mycobot_pro_600_description/urdf/link1.dae; visual mesh filename=package://mycobot_pro_600_description/urdf/link1.dae
- link link2: geometry collision mesh filename=package://mycobot_pro_600_description/urdf/link2.dae; visual mesh filename=package://mycobot_pro_600_description/urdf/link2.dae
- link link3: geometry collision mesh filename=package://mycobot_pro_600_description/urdf/link3.dae; visual mesh filename=package://mycobot_pro_600_description/urdf/link3.dae
- link link4: geometry collision mesh filename=package://mycobot_pro_600_description/urdf/link4.dae; visual mesh filename=package://mycobot_pro_600_description/urdf/link4.dae
- link link5: geometry collision mesh filename=package://mycobot_pro_600_description/urdf/link5.dae; visual mesh filename=package://mycobot_pro_600_description/urdf/link5.dae
- link link6: geometry collision mesh filename=package://mycobot_pro_600_description/urdf/link6.dae; visual mesh filename=package://mycobot_pro_600_description/urdf/link6.dae
Joints:
- added joint EndEffector: type fixed, parent link6, child endEffector, origin xyz=-0.07586 0 0 rpy=-1.57080 0 0 , axis -1 0 0
- added joint env_world_fixed_joint: type fixed, parent base, child env_world, origin xyz=-0.4 -0.0 0 rpy=0 0 0
- joint joint3_to_joint2: limit lower=-4.7123 upper=1.5708 effort=30.0 velocity=3.0 -> lower=-3.57792 upper=0.418879 effort=30.0 velocity=3.0
- joint joint4_to_joint3: limit lower=-2.6179 upper=2.443 effort=30.0 velocity=3.0 -> lower=-2.0944 upper=2.443 effort=30.0 velocity=3.0
- joint joint5_to_joint4: limit lower=-4.5378 upper=1.3962 effort=30.0 velocity=3.0 -> lower=-3.14159 upper=1.3962 effort=30.0 velocity=3.0
- joint joint6_to_joint5: limit lower=-2.9321 upper=2.9321 effort=1000.0 velocity=3.0 -> lower=-3.14 upper=3.14 effort=1000.0 velocity=3.0

Commit message: Changed Kinematics solver with Trac_Ik

File: mycobot_pro_600_description/urdf/mycobot_pro_600.urdf (robot description, URDF)
Before this commit: robot mycobot_600, 9 links, 8 joints
Links:
- link env_world: geometry collision cylinder length=0.01 radius=0.5; visual mesh filename=package://mycobot_pro_600_description/urdf/suit_env_v2.dae
Joints:
- joint EndEffector: origin xyz=-0.07586 0 0 rpy=-1.57080 0 0  -> xyz=0 0 0 rpy=-1.57080 0 0 

Commit message: merged with Rakshith and Krishna

File: mycobot_pro_600_description/urdf/mycobot_pro_600.urdf (robot description, URDF)
Before this commit: robot mycobot_600, 8 links, 7 joints
Links:
- added link endEffector
- link base: geometry collision mesh filename=package://mycobot_pro_600_description/urdf/base.dae; visual mesh filename=package://mycobot_pro_600_description/urdf/base.dae
- link env_world: geometry collision cylinder length=0.01 radius=0.5; visual mesh filename=package://mycobot_pro_600_description/urdf/suit_env_v2.dae
- link link1: geometry collision mesh filename=package://mycobot_pro_600_description/urdf/link1.dae; visual mesh filename=package://mycobot_pro_600_description/urdf/link1.dae
- link link2: geometry collision mesh filename=package://mycobot_pro_600_description/urdf/link2.dae; visual mesh filename=package://mycobot_pro_600_description/urdf/link2.dae
- link link3: geometry collision mesh filename=package://mycobot_pro_600_description/urdf/link3.dae; visual mesh filename=package://mycobot_pro_600_description/urdf/link3.dae
- link link4: geometry collision mesh filename=package://mycobot_pro_600_description/urdf/link4.dae; visual mesh filename=package://mycobot_pro_600_description/urdf/link4.dae
- link link5: geometry collision mesh filename=package://mycobot_pro_600_description/urdf/link5.dae; visual mesh filename=package://mycobot_pro_600_description/urdf/link5.dae
- link link6: geometry collision mesh filename=package://mycobot_pro_600_description/urdf/link6.dae; visual mesh filename=package://mycobot_pro_600_description/urdf/link6.dae
Joints:
- added joint EndEffector: type fixed, parent link6, child endEffector, origin xyz=0 0 0 rpy=-1.57080 0 0 , axis -1 0 0
- joint env_world_fixed_joint: origin xyz=-0.15 -0.25 0 rpy=0 0 3.14159 -> xyz=-0.15 -0.25 0 rpy=0 0 0
- joint joint3_to_joint2: limit lower=-3.14 upper=0 effort=30.0 velocity=3.0 -> lower=-3.57792 upper=0.418879 effort=30.0 velocity=3.0
- joint joint4_to_joint3: limit lower=-2.6179 upper=2.443 effort=30.0 velocity=3.0 -> lower=-2.0944 upper=2.443 effort=30.0 velocity=3.0
- joint joint5_to_joint4: limit lower=-4.5378 upper=1.3962 effort=30.0 velocity=3.0 -> lower=-3.14159 upper=1.3962 effort=30.0 velocity=3.0
- joint joint6_to_joint5: limit lower=-2.9321 upper=2.9321 effort=1000.0 velocity=3.0 -> lower=-3.14 upper=3.14 effort=1000.0 velocity=3.0

File: mycobot_pro_600_moveit_config/config/mycobot_600.urdf.xacro (robot description, xacro)
@@ -3,5 +3,5 @@
     <xacro:arg name="initial_positions_file" default="initial_positions.yaml" />
     <!-- Import mycobot_600 urdf file -->
-    <xacro:include filename="$(find mycobot_pro_600_desp)/urdf/mycobot_pro_600.urdf" />
+    <xacro:include filename="$(find mycobot_pro_600_description)/urdf/mycobot_pro_600.urdf" />
     <!-- Import control_xacro -->
     <xacro:include filename="mycobot_600.ros2_control.xacro" />

Commit message: Added waypoint control and state logging

File: mycobot_pro_600_description/urdf/mycobot_pro_600.urdf (robot description, URDF)
Before this commit: robot mycobot_600, 9 links, 8 joints
Joints:
- joint env_world_fixed_joint: origin xyz=-0.4 -0.0 0 rpy=0 0 0 -> xyz=-0.15 -0.25 0 rpy=0 0 0

Commit message: Fixed IK solution and joint rotation issues, final push for maze solver

File: mycobot_pro_600_description/urdf/mycobot_pro_600.urdf (robot description, URDF)
Before this commit: robot mycobot_600, 9 links, 8 joints
Links:
- link env_world: geometry collision cylinder length=0.02 radius=0.4; visual mesh filename=package://mycobot_pro_600_description/urdf/suit_env_v2.dae
Joints:
- joint env_world_fixed_joint: origin xyz=-0.15 -0.25 0 rpy=0 0 0 -> xyz=-0.25 0.0 0 rpy=0 0 0
- joint joint2_to_joint1: limit lower=-3.14 upper=3.14159 effort=30.0 velocity=3.0 -> lower=-1.97 upper=0.43 effort=30.0 velocity=3.0
- joint joint3_to_joint2: limit lower=-3.57792 upper=0.418879 effort=30.0 velocity=3.0 -> lower=-3.14 upper=0 effort=30.0 velocity=3.0
- joint joint4_to_joint3: limit lower=-2.0944 upper=2.443 effort=30.0 velocity=3.0 -> lower=-3.14 upper=3.14 effort=30.0 velocity=3.0
- joint joint5_to_joint4: limit lower=-3.14159 upper=1.3962 effort=30.0 velocity=3.0 -> lower=-3.14 upper=3.14 effort=30.0 velocity=3.0
- joint joint6output_to_joint6: limit lower=-3.0368 upper=3.0368 effort=30.0 velocity=3.0 -> lower=-3.14 upper=3.14 effort=30.0 velocity=3.0
